Commit message: change packag ename dvrk_model2

File: dvrk_model2/deprecated/urdf/daVinci_jhu.urdf (robot description, URDF)
Before this commit: robot daVinci, 14 links, 13 joints
Links:
- link outer_insertion_link: geometry visual mesh filename=package://dvrk_model2/meshes/outer_insertion.dae
- link outer_pitch_back_link: geometry visual mesh filename=package://dvrk_model2/meshes/outer_pitch_back.dae
- link outer_pitch_bottom_link: geometry visual mesh filename=package://dvrk_model2/meshes/outer_pitch_bottom.dae
- link outer_pitch_front_link: geometry visual mesh filename=package://dvrk_model2/meshes/outer_pitch_front.dae
- link outer_pitch_top_link: geometry visual mesh filename=package://dvrk_model2/meshes/outer_pitch_top.dae
- link outer_yaw_link: geometry visual mesh filename=package://dvrk_model2/meshes/outer_yaw.dae
- link psm_base_link: geometry visual mesh filename=package://dvrk_model2/meshes/psm_base.dae
- link tool_main_link: geometry visual mesh filename=package://dvrk_model2/meshes/tool_main.dae
- link tool_wrist_link: geometry visual mesh filename=package://dvrk_model2/meshes/tool_wrist_link.dae
- link tool_wrist_sca_ee_link_1: geometry visual mesh filename=package://dvrk_model2/meshes/tool_wrist_sca_link_2.dae
- link tool_wrist_sca_ee_link_2: geometry visual mesh filename=package://dvrk_model2/meshes/tool_wrist_sca_link_2.dae
- link tool_wrist_sca_link: geometry visual mesh filename=package://dvrk_model2/meshes/tool_wrist_sca_link.dae
- link tool_wrist_sca_shaft_link: geometry visual mesh filename=package://dvrk_model2/meshes/tool_wrist_sca_shaft_link.dae
- link tool_wrist_shaft_link: geometry visual mesh filename=package://dvrk_model2/meshes/tool_wrist_shaft_link.dae

File: dvrk_model2/model/ECM.urdf.xacro (robot description, xacro)
@@ -2,5 +2,5 @@
 <robot name="ecm" xmlns:xacro="http://www.ros.org/wiki/xacro">
   <!-- Macros -->
-  <xacro:include filename="$(find dvrk_model)/model/ecm.urdf.xacro"/>
+  <xacro:include filename="$(find dvrk_model2)/model/ecm.urdf.xacro"/>
   <link name="world"/>
   <xacro:ecm

File: dvrk_model2/model/MTML.urdf.xacro (robot description, xacro)
@@ -2,5 +2,5 @@
 <robot name="master" xmlns:xacro="http://www.ros.org/wiki/xacro">
   <!-- Macros -->
-  <xacro:include filename="$(find dvrk_model)/model/mtm.urdf.xacro"/>
+  <xacro:include filename="$(find dvrk_model2)/model/mtm.urdf.xacro"/>
   <link name="world"/>
   <xacro:mtm_left

File: dvrk_model2/model/MTMR.urdf.xacro (robot description, xacro)
@@ -2,5 +2,5 @@
 <robot name="master" xmlns:xacro="http://www.ros.org/wiki/xacro">
   <!-- Macros -->
-  <xacro:include filename="$(find dvrk_model)/model/mtm.urdf.xacro"/>
+  <xacro:include filename="$(find dvrk_model2)/model/mtm.urdf.xacro"/>
   <link name="world"/>
   <xacro:mtm_right

File: dvrk_model2/model/PSM1.urdf.xacro (robot description, xacro)
@@ -2,9 +2,9 @@
 <robot name="dvrk_psm" xmlns:xacro="http://www.ros.org/wiki/xacro">
   <!-- Macros -->
-  <xacro:include filename="$(find dvrk_model)/model/psm.urdf.xacro"/>
+  <xacro:include filename="$(find dvrk_model2)/model/psm.urdf.xacro"/>
   <link name="world"/>
-  <xacro:psm_caudier
+  <xacro:psm_sca
       prefix="$(arg prefix)"
       parent_link="world"
-      xyz="0.25 0.0 0.5" rpy="0.0 0.0 -3.1415926"/>
+      xyz="-0.25 0.0 0.5" rpy="0.0 0.0 3.1415926"/>
 </robot>

File: dvrk_model2/model/PSM2.urdf.xacro (robot description, xacro)
@@ -2,9 +2,9 @@
 <robot name="dvrk_psm" xmlns:xacro="http://www.ros.org/wiki/xacro">
   <!-- Macros -->
-  <xacro:include filename="$(find dvrk_model)/model/psm.urdf.xacro"/>
+  <xacro:include filename="$(find dvrk_model2)/model/psm.urdf.xacro"/>
   <link name="world"/>
-  <xacro:psm_sca
+  <xacro:psm_caudier
       prefix="$(arg prefix)"
       parent_link="world"
-      xyz="-0.25 0.0 0.5" rpy="0.0 0.0 3.1415926"/>
+      xyz="0.25 0.0 0.5" rpy="0.0 0.0 -3.1415926"/>
 </robot>

File: dvrk_model2/model/PSM3.urdf.xacro (robot description, xacro)
@@ -2,5 +2,5 @@
 <robot name="dvrk_psm" xmlns:xacro="http://www.ros.org/wiki/xacro">
   <!-- Macros -->
-  <xacro:include filename="$(find dvrk_model)/model/psm.urdf.xacro"/>
+  <xacro:include filename="$(find dvrk_model2)/model/psm.urdf.xacro"/>
   <link name="world"/>
   <xacro:psm_caudier

File: dvrk_model2/model/both_psms.urdf.xacro (robot description, xacro)
@@ -2,5 +2,5 @@
 <robot name="dvrk_psm" xmlns:xacro="http://www.ros.org/wiki/xacro">
   <!-- Macros -->
-  <xacro:include filename="$(find dvrk_model)/model/psm.urdf.xacro"/>
+  <xacro:include filename="$(find dvrk_model2)/model/psm.urdf.xacro"/>
   <link name="world">
       <origin xyz="0.0 0.0 0.0"/>

File: dvrk_model2/model/ecm.urdf.xacro (robot description, xacro)
@@ -2,5 +2,5 @@
 <robot name="ecm" xmlns:xacro="http://www.ros.org/wiki/xacro">
   <!-- Colors -->
-  <xacro:include filename="$(find dvrk_model)/model/common.urdf.xacro"/>
+  <xacro:include filename="$(find dvrk_model2)/model/common.urdf.xacro"/>
   <!-- Macro for da Vinci Endoscope Camera Manipulator (ECM) -->
   <xacro:macro name="ecm" params="prefix parent_link xyz rpy">

File: dvrk_model2/model/mtm.urdf.xacro (robot description, xacro)
@@ -2,5 +2,5 @@
 <robot name="mtm" xmlns:xacro="http://www.ros.org/wiki/xacro">
   <!-- Colors -->
-  <xacro:include filename="$(find dvrk_model)/model/common.urdf.xacro"/>
+  <xacro:include filename="$(find dvrk_model2)/model/common.urdf.xacro"/>
   <!-- Macro for the da Vinci Master Console -->
   <xacro:macro name="master_console" params="prefix parent_link xyz rpy">

File: dvrk_model2/model/psm.base.urdf.xacro (robot description, xacro)
@@ -13,5 +13,5 @@
         <origin rpy="1.5708 0 3.1416" xyz="0.039 -0.40788 -0.07879"/>
         <geometry>
-          <mesh filename="package://dvrk_model/meshes/psm/psm_base.dae"/>
+          <mesh filename="package://dvrk_model2/meshes/psm/psm_base.dae"/>
         </geometry>
       </visual>
@@ -31,5 +31,5 @@
         <origin rpy="3.1416 0 1.5708" xyz="0.0125 0 0.5265"/>
         <geometry>
-          <mesh filename="package://dvrk_model/meshes/psm/outer_yaw.dae"/>
+          <mesh filename="package://dvrk_model2/meshes/psm/outer_yaw.dae"/>
         </geometry>
       </visual>
@@ -62,5 +62,5 @@
         <origin rpy="0 0 -0.27129" xyz="0 0 0"/>
         <geometry>
-          <mesh filename="package://dvrk_model/meshes/psm/outer_pitch_back.dae"/>
+          <mesh filename="package://dvrk_model2/meshes/psm/outer_pitch_back.dae"/>
         </geometry>
       </visual>
@@ -79,5 +79,5 @@
         <origin rpy="0 0 -0.27129" xyz="0 0 0"/>
         <geometry>
-          <mesh filename="package://dvrk_model/meshes/psm/outer_pitch_front.dae"/>
+          <mesh filename="package://dvrk_model2/meshes/psm/outer_pitch_front.dae"/>
         </geometry>
       </visual>
@@ -96,5 +96,5 @@
         <origin rpy="0 -1.5708 0" xyz="0.009 0 0"/>
         <geometry>
-          <mesh filename="package://dvrk_model/meshes/psm/outer_pitch_bottom.dae"/>
+          <mesh filename="package://dvrk_model2/meshes/psm/outer_pitch_bottom.dae"/>
         </geometry>
       </visual>
@@ -113,5 +113,5 @@
         <origin rpy="0 -1.5708 0" xyz="0.009 0 0"/>
         <geometry>
-          <mesh filename="package://dvrk_model/meshes/psm/outer_pitch_top.dae"/>
+          <mesh filename="package://dvrk_model2/meshes/psm/outer_pitch_top.dae"/>
         </geometry>
       </visual>
@@ -130,5 +130,5 @@
         <origin rpy="0 -1.5708 1.5708" xyz="0.02528 0.429 0"/>
         <geometry>
-          <mesh filename="package://dvrk_model/meshes/psm/outer_insertion.dae"/>
+          <mesh filename="package://dvrk_model2/meshes/psm/outer_insertion.dae"/>
         </geometry>
       </visual>
@@ -149,5 +149,5 @@
         <origin rpy="0 0 1.5708" xyz="0 0 0.041"/>
         <geometry>
-          <mesh filename="package://dvrk_model/meshes/psm/tool_main.dae"/>
+          <mesh filename="package://dvrk_model2/meshes/psm/tool_main.dae"/>
         </geometry>
       </visual>
@@ -166,5 +166,5 @@
         <origin rpy="0 0 1.5708" xyz="0 0 -0.0091"/>
         <geometry>
-          <mesh filename="package://dvrk_model/meshes/psm/tool_wrist_link.dae"/>
+          <mesh filename="package://dvrk_model2/meshes/psm/tool_wrist_link.dae"/>
         </geometry>
       </visual>
@@ -182,5 +182,5 @@
         <origin rpy="1.5708 0 0" xyz="0 0.00401 0"/>
         <geometry>
-          <mesh filename="package://dvrk_model/meshes/psm/tool_wrist_shaft_link.dae"/>
+          <mesh filename="package://dvrk_model2/meshes/psm/tool_wrist_shaft_link.dae"/>
         </geometry>
       </visual>

File: dvrk_model2/model/psm.tool.caudier.urdf.xacro (robot description, xacro)
@@ -15,5 +15,5 @@
         <origin rpy="0.00 -1.5708 0.0" xyz="-0.0024 0.00 0.000"/>
         <geometry>
-          <mesh filename="package://dvrk_model/meshes/psm/tool_wrist_caudier_link_1.stl"/>
+          <mesh filename="package://dvrk_model2/meshes/psm/tool_wrist_caudier_link_1.stl"/>
         </geometry>
         <material name="gray"><color rgba="0.5 0.5 0.9 1.0"/></material>
@@ -22,5 +22,5 @@
         <origin rpy="0.00 -1.5708 0.0" xyz="-0.0024 0.00 0.000"/>
         <geometry>
-          <mesh filename="package://dvrk_model/meshes/psm/tool_wrist_caudier_link_1.stl"/>
+          <mesh filename="package://dvrk_model2/meshes/psm/tool_wrist_caudier_link_1.stl"/>
         </geometry>
       </collision>
@@ -39,5 +39,5 @@
         <origin rpy="0.00 1.5708 0.0" xyz="0.0 -0.0002 0.000"/>
         <geometry>
-          <mesh filename="package://dvrk_model/meshes/psm/tool_wrist_caudier_link_1_shaft.stl"/>
+          <mesh filename="package://dvrk_model2/meshes/psm/tool_wrist_caudier_link_1_shaft.stl"/>
         </geometry>
         <material name="gray"><color rgba="0.5 0.5 0.9 1.0"/></material>
@@ -46,5 +46,5 @@
         <origin rpy="0.00 1.5708 0.0" xyz="0.0 0.00 0.000"/>
         <geometry>
-          <mesh filename="package://dvrk_model/meshes/psm/tool_wrist_caudier_link_1_shaft.stl"/>
+          <mesh filename="package://dvrk_model2/meshes/psm/tool_wrist_caudier_link_1_shaft.stl"/>
         </geometry>
       </collision>
@@ -81,5 +81,5 @@
         <origin rpy="0.0 0 0.0" xyz="0 0 0.00195"/>
         <geometry>
-          <mesh filename="package://dvrk_model/meshes/psm/tool_wrist_caudier_link_2.stl"/>
+          <mesh filename="package://dvrk_model2/meshes/psm/tool_wrist_caudier_link_2.stl"/>
         </geometry>
       </visual>
@@ -99,5 +99,5 @@
         <origin rpy="0 0 -3.1415926" xyz="0 0 0.00195"/>
         <geometry>
-          <mesh filename="package://dvrk_model/meshes/psm/tool_wrist_caudier_link_2.stl"/>
+          <mesh filename="package://dvrk_model2/meshes/psm/tool_wrist_caudier_link_2.stl"/>
         </geometry>
       </visual>

File: dvrk_model2/model/psm.tool.sca.urdf.xacro (robot description, xacro)
@@ -2,5 +2,5 @@
 <robot name="dvrk_psm" xmlns:xacro="http://www.ros.org/wiki/xacro">
   <!-- This file contains different tool urdf -->
-  <xacro:include filename="$(find dvrk_model)/model/common.urdf.xacro"/>
+  <xacro:include filename="$(find dvrk_model2)/model/common.urdf.xacro"/>
   <!-- sca  -->
   <xacro:macro name="psm_tool_sca" params="prefix">
@@ -19,5 +19,5 @@
         <origin rpy="1.5708 3.1416 0" xyz="0.0051 0.0032 0"/>
         <geometry>
-          <mesh filename="package://dvrk_model/meshes/psm/tool_wrist_sca_link.dae"/>
+          <mesh filename="package://dvrk_model2/meshes/psm/tool_wrist_sca_link.dae"/>
         </geometry>
       </visual>
@@ -37,5 +37,5 @@
         <origin rpy="0 0 0" xyz="0 -0.0002 -0.0025"/>
         <geometry>
-          <mesh filename="package://dvrk_model/meshes/psm/tool_wrist_sca_shaft_link.dae"/>
+          <mesh filename="package://dvrk_model2/meshes/psm/tool_wrist_sca_shaft_link.dae"/>
         </geometry>
       </visual>
@@ -72,5 +72,5 @@
         <origin rpy="0 0 0" xyz="0 0 0"/>
         <geometry>
-          <mesh filename="package://dvrk_model/meshes/psm/tool_wrist_sca_link_2.dae"/>
+          <mesh filename="package://dvrk_model2/meshes/psm/tool_wrist_sca_link_2.dae"/>
         </geometry>
       </visual>
@@ -90,5 +90,5 @@
         <origin rpy="0 3.1516 0" xyz="0 0 0"/>
         <geometry>
-          <mesh filename="package://dvrk_model/meshes/psm/tool_wrist_sca_link_2.dae"/>
+          <mesh filename="package://dvrk_model2/meshes/psm/tool_wrist_sca_link_2.dae"/>
         </geometry>
       </visual>

File: dvrk_model2/model/psm.urdf.xacro (robot description, xacro)
@@ -2,7 +2,7 @@
 <robot name="dvrk_psm" xmlns:xacro="http://www.ros.org/wiki/xacro">
   <!-- Macros -->
-  <xacro:include filename="$(find dvrk_model)/model/psm.base.urdf.xacro"/>
-  <xacro:include filename="$(find dvrk_model)/model/psm.tool.sca.urdf.xacro"/>
-  <xacro:include filename="$(find dvrk_model)/model/psm.tool.caudier.urdf.xacro"/>
+  <xacro:include filename="$(find dvrk_model2)/model/psm.base.urdf.xacro"/>
+  <xacro:include filename="$(find dvrk_model2)/model/psm.tool.sca.urdf.xacro"/>
+  <xacro:include filename="$(find dvrk_model2)/model/psm.tool.caudier.urdf.xacro"/>
   <!-- Macro for psm with sca -->
   <xacro:macro name="psm_sca" params="prefix parent_link xyz rpy">
