Commit message: change package name dvrk_model2

File: dvrk_model2/model/ecm.urdf.xacro (robot description, xacro)
@@ -22,5 +22,5 @@
         <origin rpy="0 0 0" xyz="0 0 0"/>
         <geometry>
-          <mesh filename="package://dvrk_model/meshes/ecm/Endo_Arm.STL"/>
+          <mesh filename="package://dvrk_model2/meshes/ecm/Endo_Arm.STL"/>
         </geometry>
 	<material name="DaVinciRed"/>
@@ -29,5 +29,5 @@
         <origin rpy="0 0 0" xyz="0 0 0"/>
         <geometry>
-          <mesh filename="package://dvrk_model/meshes/ecm/Endo_Arm.STL"/>
+          <mesh filename="package://dvrk_model2/meshes/ecm/Endo_Arm.STL"/>
         </geometry>
       </collision>
@@ -55,5 +55,5 @@
         <origin rpy="0 0 -${PI/2}" xyz="0.0 0 0.603"/>
         <geometry>
-          <mesh filename="package://dvrk_model/meshes/ecm/Endo_Link_5.STL"/>
+          <mesh filename="package://dvrk_model2/meshes/ecm/Endo_Link_5.STL"/>
         </geometry>
 	<material name="DaVinciGreen"/>
@@ -62,5 +62,5 @@
         <origin rpy="0 0 -${PI/2}" xyz="0.0 0 0.603"/>
         <geometry>
-          <mesh filename="package://dvrk_model/meshes/ecm/Endo_Link_5.STL"/>
+          <mesh filename="package://dvrk_model2/meshes/ecm/Endo_Link_5.STL"/>
         </geometry>
       </collision>
@@ -88,5 +88,5 @@
         <origin rpy="${PI} 0 ${PI*78.5/180}" xyz="0.0 0 0.0"/>
         <geometry>
-          <mesh filename="package://dvrk_model/meshes/ecm/Endo_Link_5_2.STL"/>
+          <mesh filename="package://dvrk_model2/meshes/ecm/Endo_Link_5_2.STL"/>
         </geometry>
 	<material name="DaVinciMedGray"/>
@@ -95,5 +95,5 @@
         <origin rpy="${PI} 0 ${PI*78.5/180}" xyz="0.0 0 0.0"/>
         <geometry>
-          <mesh filename="package://dvrk_model/meshes/ecm/Endo_Link_5_2.STL"/>
+          <mesh filename="package://dvrk_model2/meshes/ecm/Endo_Link_5_2.STL"/>
         </geometry>
       </collision>
@@ -115,5 +115,5 @@
         <origin rpy="0 0 0" xyz="0.0 0 -0.0225"/>
         <geometry>
-          <mesh filename="package://dvrk_model/meshes/ecm/Endo_Link_6_2.STL"/>
+          <mesh filename="package://dvrk_model2/meshes/ecm/Endo_Link_6_2.STL"/>
         </geometry>
 	<material name="DaVinciMedGray"/>
@@ -122,5 +122,5 @@
         <origin rpy="0 0 0" xyz="0.0 0 -0.0225"/>
         <geometry>
-          <mesh filename="package://dvrk_model/meshes/ecm/Endo_Link_6_2.STL"/>
+          <mesh filename="package://dvrk_model2/meshes/ecm/Endo_Link_6_2.STL"/>
         </geometry>
       </collision>
@@ -142,5 +142,5 @@
         <origin rpy="0 0 -${PI/2}" xyz="0.0 0 0.025"/>
         <geometry>
-          <mesh filename="package://dvrk_model/meshes/ecm/Endo_Link_7.STL"/>
+          <mesh filename="package://dvrk_model2/meshes/ecm/Endo_Link_7.STL"/>
         </geometry>
 	<material name="DaVinciMedGray"/>
@@ -149,5 +149,5 @@
         <origin rpy="0 0 -${PI/2}" xyz="0.0 0 0.025"/>
         <geometry>
-          <mesh filename="package://dvrk_model/meshes/ecm/Endo_Link_7.STL"/>
+          <mesh filename="package://dvrk_model2/meshes/ecm/Endo_Link_7.STL"/>
         </geometry>
       </collision>
@@ -170,5 +170,5 @@
         <origin rpy="0 0 -${PI/2}" xyz="0.0 0 -0.015"/>
         <geometry>
-          <mesh filename="package://dvrk_model/meshes/ecm/Endo_Link_8.STL"/>
+          <mesh filename="package://dvrk_model2/meshes/ecm/Endo_Link_8.STL"/>
         </geometry>
 	<material name="DaVinciBlue"/>
@@ -177,5 +177,5 @@
         <origin rpy="0 0 -${PI/2}" xyz="0.0 0 -0.015"/>
         <geometry>
-          <mesh filename="package://dvrk_model/meshes/ecm/Endo_Link_8.STL"/>
+          <mesh filename="package://dvrk_model2/meshes/ecm/Endo_Link_8.STL"/>
         </geometry>
       </collision>
@@ -194,5 +194,5 @@
         <origin rpy="0 0 ${PI/2}" xyz="0.0 0 -0.3979"/>
         <geometry>
-          <mesh filename="package://dvrk_model/meshes/ecm/EndoScope.STL"/>
+          <mesh filename="package://dvrk_model2/meshes/ecm/EndoScope.STL"/>
         </geometry>
 	<material name="DaVinciBlue"/>
@@ -201,5 +201,5 @@
         <origin rpy="0 0 ${PI/2}" xyz="0.0 0 -0.3979"/>
         <geometry>
-          <mesh filename="package://dvrk_model/meshes/ecm/EndoScope.STL"/>
+          <mesh filename="package://dvrk_model2/meshes/ecm/EndoScope.STL"/>
         </geometry>
       </collision>

File: dvrk_model2/model/mtm.urdf.xacro (robot description, xacro)
@@ -41,5 +41,5 @@
         <origin rpy="0 0 0" xyz="0 0 0.19037"/>
         <geometry>
-          <mesh filename="package://dvrk_model/meshes/mtm/Top Panel.dae"/>
+          <mesh filename="package://dvrk_model2/meshes/mtm/Top Panel.dae"/>
         </geometry>
       </visual>
@@ -47,5 +47,5 @@
         <origin rpy="0 0 0" xyz="0 0 0.19037"/>
         <geometry>
-          <mesh filename="package://dvrk_model/meshes/mtm/Top Panel.STL"/>
+          <mesh filename="package://dvrk_model2/meshes/mtm/Top Panel.STL"/>
         </geometry>
       </collision>
@@ -73,5 +73,5 @@
         <origin rpy="0 0 0" xyz="0.025 0 0.19037"/>
         <geometry>
-          <mesh filename="package://dvrk_model/meshes/mtm/OutPitch_Shoulder.dae"/>
+          <mesh filename="package://dvrk_model2/meshes/mtm/OutPitch_Shoulder.dae"/>
         </geometry>
       </visual>
@@ -79,5 +79,5 @@
         <origin rpy="0 0 0" xyz="0.025 0 0.19037"/>
         <geometry>
-          <mesh filename="package://dvrk_model/meshes/mtm/OutPitch_Shoulder.STL"/>
+          <mesh filename="package://dvrk_model2/meshes/mtm/OutPitch_Shoulder.STL"/>
         </geometry>
       </collision>
@@ -100,10 +100,10 @@
       <visual>
         <geometry>
-          <mesh filename="package://dvrk_model/meshes/mtm/ArmParallel.dae"/>
-        </geometry>
-      </visual>
-      <collision>
-        <geometry>
-          <mesh filename="package://dvrk_model/meshes/mtm/ArmParallel.STL"/>
+          <mesh filename="package://dvrk_model2/meshes/mtm/ArmParallel.dae"/>
+        </geometry>
+      </visual>
+      <collision>
+        <geometry>
+          <mesh filename="package://dvrk_model2/meshes/mtm/ArmParallel.STL"/>
         </geometry>
       </collision>
@@ -128,5 +128,5 @@
         <origin rpy="0 0 ${-PI/2}" xyz="0 0 0.065"/>
         <geometry>
-          <mesh filename="package://dvrk_model/meshes/mtm/ArmParallel1.dae"/>
+          <mesh filename="package://dvrk_model2/meshes/mtm/ArmParallel1.dae"/>
         </geometry>
       </visual>
@@ -134,5 +134,5 @@
         <origin rpy="0 0 0" xyz="0 0 0"/>
         <geometry>
-          <mesh filename="package://dvrk_model/meshes/mtm/ArmParallel1.STL"/>
+          <mesh filename="package://dvrk_model2/meshes/mtm/ArmParallel1.STL"/>
         </geometry>
       </collision>
@@ -155,10 +155,10 @@
       <visual>
         <geometry>
-          <mesh filename="package://dvrk_model/meshes/mtm/BottomArm.dae"/>
-        </geometry>
-      </visual>
-      <collision>
-        <geometry>
-          <mesh filename="package://dvrk_model/meshes/mtm/BottomArm.STL"/>
+          <mesh filename="package://dvrk_model2/meshes/mtm/BottomArm.dae"/>
+        </geometry>
+      </visual>
+      <collision>
+        <geometry>
+          <mesh filename="package://dvrk_model2/meshes/mtm/BottomArm.STL"/>
         </geometry>
       </collision>
@@ -225,10 +225,10 @@
       <visual>
         <geometry>
-          <mesh filename="package://dvrk_model/meshes/mtm/WristPlatform.dae"/>
-        </geometry>
-      </visual>
-      <collision>
-        <geometry>
-          <mesh filename="package://dvrk_model/meshes/mtm/WristPlatform.STL"/>
+          <mesh filename="package://dvrk_model2/meshes/mtm/WristPlatform.dae"/>
+        </geometry>
+      </visual>
+      <collision>
+        <geometry>
+          <mesh filename="package://dvrk_model2/meshes/mtm/WristPlatform.STL"/>
         </geometry>
       </collision>
@@ -253,10 +253,10 @@
       <visual>        <!-- defined from CAD file (increased in the y dir by .005-->
         <geometry>
-          <mesh filename="package://dvrk_model/meshes/mtm/WristPitch.dae"/>
+          <mesh filename="package://dvrk_model2/meshes/mtm/WristPitch.dae"/>
         </geometry>
       </visual>
       <collision>        <!-- defined from CAD file (increased in the y dir by .005-->
         <geometry>
-          <mesh filename="package://dvrk_model/meshes/mtm/WristPitch.STL"/>
+          <mesh filename="package://dvrk_model2/meshes/mtm/WristPitch.STL"/>
         </geometry>
       </collision>
@@ -282,10 +282,10 @@
       <visual>
         <geometry>
-          <mesh filename="package://dvrk_model/meshes/mtm/WristYaw.dae"/>
-        </geometry>
-      </visual>
-      <collision>
-        <geometry>
-          <mesh filename="package://dvrk_model/meshes/mtm/WristYaw.STL"/>
+          <mesh filename="package://dvrk_model2/meshes/mtm/WristYaw.dae"/>
+        </geometry>
+      </visual>
+      <collision>
+        <geometry>
+          <mesh filename="package://dvrk_model2/meshes/mtm/WristYaw.STL"/>
         </geometry>
       </collision>
@@ -312,5 +312,5 @@
         <origin rpy="${PI} 0 0" xyz="0 0 0.039"/>
         <geometry>
-          <mesh filename="package://dvrk_model/meshes/mtm/WristRoll.dae"/>
+          <mesh filename="package://dvrk_model2/meshes/mtm/WristRoll.dae"/>
         </geometry>
       </visual>
@@ -318,5 +318,5 @@
         <origin rpy="${PI} 0 0" xyz="0 0 0.039"/>
         <geometry>
-          <mesh filename="package://dvrk_model/meshes/mtm/WristRoll.STL"/>
+          <mesh filename="package://dvrk_model2/meshes/mtm/WristRoll.STL"/>
         </geometry>
       </collision>
@@ -378,5 +378,5 @@
         <origin rpy="0 0 ${PI}" xyz="0.0 0.0 0.0"/>
         <geometry>
-          <mesh filename="package://dvrk_model/meshes/mtm/WristPlatform.dae"/>
+          <mesh filename="package://dvrk_model2/meshes/mtm/WristPlatform.dae"/>
         </geometry>
       </visual>
@@ -384,5 +384,5 @@
         <origin rpy="0 0 ${PI}" xyz="0.0 0.0 0.0"/>
         <geometry>
-          <mesh filename="package://dvrk_model/meshes/mtm/WristPlatform.STL"/>
+          <mesh filename="package://dvrk_model2/meshes/mtm/WristPlatform.STL"/>
         </geometry>
       </collision>
@@ -408,5 +408,5 @@
         <origin rpy="0 ${PI} 0" xyz="0.0 0.0 0.0"/>
         <geometry>
-          <mesh filename="package://dvrk_model/meshes/mtm/WristPitch.dae"/>
+          <mesh filename="package://dvrk_model2/meshes/mtm/WristPitch.dae"/>
         </geometry>
       </visual>
@@ -414,5 +414,5 @@
         <origin rpy="0 ${PI} 0" xyz="0.0 0.0 0.0"/>
         <geometry>
-          <mesh filename="package://dvrk_model/meshes/mtm/WristPitch.STL"/>
+          <mesh filename="package://dvrk_model2/meshes/mtm/WristPitch.STL"/>
         </geometry>
       </collision>
@@ -438,10 +438,10 @@
       <visual>
         <geometry>
-          <mesh filename="package://dvrk_model/meshes/mtm/WristYaw.dae"/>
-        </geometry>
-      </visual>
-      <collision>
-        <geometry>
-          <mesh filename="package://dvrk_model/meshes/mtm/WristYaw.STL"/>
+          <mesh filename="package://dvrk_model2/meshes/mtm/WristYaw.dae"/>
+        </geometry>
+      </visual>
+      <collision>
+        <geometry>
+          <mesh filename="package://dvrk_model2/meshes/mtm/WristYaw.STL"/>
         </geometry>
       </collision>
@@ -468,5 +468,5 @@
         <origin rpy="${PI} 0 0" xyz="0 0 0.039"/>
         <geometry>
-          <mesh filename="package://dvrk_model/meshes/mtm/WristRoll.dae"/>
+          <mesh filename="package://dvrk_model2/meshes/mtm/WristRoll.dae"/>
         </geometry>
       </visual>
@@ -474,5 +474,5 @@
         <origin rpy="${PI} 0 0" xyz="0 0 0.039"/>
         <geometry>
-          <mesh filename="package://dvrk_model/meshes/mtm/WristRoll.STL"/>
+          <mesh filename="package://dvrk_model2/meshes/mtm/WristRoll.STL"/>
         </geometry>
       </collision>
